File: Hardware/Time-O-Mat_SegmentDisplay/Time-O-Mat_SegmentDisplay_H00/Time-O-Mat_SegmentDisplay_H00.kicad_pcb (KiCad board)
At the start: 2 copper layers, 55.1 x 132.3 mm, 49 parts, among them J1 Conn_02x04_Odd_Even

Commit message: Colon update
Parts:
- added G1: Vedatori_logo, Time-O-Mat_Library:Vedatori_15mm, B.Cu at (0.00, 0.00)
- added G2: CoufalElektronika_logo, Time-O-Mat_Library:Coufal_elektronika_notext_10mm, B.Cu at (0.00, 76.2)
Other:
- board text added: "Time-O-Mat_SegmentDisplay_H00"
