File: Hardware/Time-O-Mat_SegmentDisplay/Time-O-Mat_SegmentDisplay_H00/_autosave-Time-O-Mat_SegmentDisplay_H00.kicad_pcb (KiCad board)
At the start: 2 copper layers, 55.1 x 132.3 mm, 49 parts, among them J1 Conn_02x04_Odd_Even

Commit message: PCB updates
Other:
- board text added: "Time-O-Mat_SegmentDisplay_H00"
Changed lines of the file:
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@@
   (gr_line (start 18.565685 -4.5) (end 18.565685 -41.631371) (layer "Edge.Cuts") (width 0.1))
   (gr_line (start 18.565685 41.631371) (end -18.565685 41.631371) (layer "Edge.Cuts") (width 0.1))
+  (gr_text "Time-O-Mat_SegmentDisplay_H00" (at 0 55.9) (layer "F.SilkS")
+    (effects (font (size 1 1) (thickness 0.15)))
+  )
   (segment (start -6.581371 -47.731371) (end -10.55 -47.731371) (width 0.254) (layer "F.Cu") (net 1))
   (segment (start -3.381371 -44.531371) (end -6.581371 -47.731371) (width 0.254) (layer "F.Cu") (net 1))
