File: Hardware/Time-O-Mat_Colon/Time-O-Mat_Colon_H00/Time-O-Mat_Colon_H00.kicad_sch (KiCad schematic)
At the start: 51 parts, among them J1 Conn_02x04_Odd_Even

Commit message: Colon update
Parts:
- removed C10, C11, C12, C13, C14, C15, C16, C17, C18, C19, C20, C21, C3, C4, C5, C6, C7, C8, C9: 100nF, Capacitor_SMD:C_0402_1005Metric, symbol Device:C
- removed D10, D11, D12, D13, D14, D15, D16, D17, D18, D19, D20, D21, D3, D4, D5, D6, D7, D8, D9: WS2812E, LED_SMD:LED_WS2812B_PLCC4_5.0x5.0mm_P3.2mm, symbol LED:WS2812B
Connections:
- net at J1.5 (Pin_5), J1.6 (Pin_6): now also D2.2 (DOUT)
