File: Hardware/Time-O-Mat_TouchBar/Time-O-Mat_TouchBar_H00/Time-O-Mat_TouchBar_H00.kicad_pcb (KiCad board)
At the start: 2 copper layers, 1 part, among them J1 Conn_01x06_Male

Commit message: HW updates
Parts:
- moved J1 103.8 mm to (14.0, 8.00)
Routing:
- net TOUCH5: track 0.00 -> 72.5 mm, vias 0 -> 1
- net TOUCH6: track 0.00 -> 50.5 mm, vias 0 -> 1
- net TOUCH7: track 0.00 -> 29.5 mm, vias 0 -> 1
- net TOUCH9: track 23.6 -> 0.00 mm
- net TOUCH8: track 0.00 -> 9.56 mm, vias 0 -> 1
- net GND: track 0.00 -> 5.41 mm, vias 0 -> 1
- added copper zone on F.Cu, net TOUCH5
- added copper zone on F.Cu, net TOUCH6
- added copper zone on F.Cu, net TOUCH7
- added copper zone on F.Cu, net TOUCH8
- removed copper zone on F.Cu, net GND
Other:
- board outline added: 120 x 10 mm
Changed lines of the file:
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@@
   )
   (setup
+    (stackup
+      (layer "F.SilkS" (type "Top Silk Screen"))
+      (layer "F.Paste" (type "Top Solder Paste"))
+      (layer "F.Mask" (type "Top Solder Mask") (thickness 0.01))
+      (layer "F.Cu" (type "copper") (thickness 0.035))
+      (layer "dielectric 1" (type "core") (thickness 1.51) (material "FR4") (epsilon_r 4.5) (loss_tangent 0.02))
+      (layer "B.Cu" (type "copper") (thickness 0.035))
+      (layer "B.Mask" (type "Bottom Solder Mask") (thickness 0.01))
+      (layer "B.Paste" (type "Bottom Solder Paste"))
+      (layer "B.SilkS" (type "Bottom Silk Screen"))
+      (copper_finish "None")
+      (dielectric_constraints no)
+    )
     (pad_to_mask_clearance 0)
     (pcbplotparams
@@
   (net 6 "GND")
   (footprint "Connector_PinHeader_2.54mm:PinHeader_1x06_P2.54mm_Vertical" (layer "B.Cu")
-    (at 94.92 73 -90)
+    (at 14 8 -90)
     (descr "Through hole straight pin header, 1x06, 2.54mm pitch, single row")
     (tags "Through hole pin header THT 1x06 2.54mm single row")
@@
     )
   )
-  (segment (start 94.92 73) (end 100.92 67) (width 0.25) (layer "F.Cu") (net 1))
-  (segment (start 100.92 67) (end 116 67) (width 0.25) (layer "F.Cu") (net 1))
+  (gr_line (start 0 0) (end 0 10) (layer "Edge.Cuts") (width 0.1))
+  (gr_line (start 0 10) (end 120 10) (layer "Edge.Cuts") (width 0.1))
+  (gr_line (start 120 0) (end 0 0) (layer "Edge.Cuts") (width 0.1))
+  (gr_line (start 120 10) (end 120 0) (layer "Edge.Cuts") (width 0.1))
+  (via (at 25 5.334) (size 0.8) (drill 0.4) (layers "F.Cu" "B.Cu") (net 2))
+  (segment (start 18.71604 5.82396) (end 16.54 8) (width 0.127) (layer "B.Cu") (net 2))
+  (segment (start 25 5.334) (end 24.51004 5.82396) (width 0.127) (layer "B.Cu") (net 2))
+  (segment (start 24.51004 5.82396) (end 18.71604 5.82396) (width 0.127) (layer "B.Cu") (net 2))
+  (via (at 46.736 7.366) (size 0.8) (drill 0.4) (layers "F.Cu" "B.Cu") (net 3))
+  (segment (start 20.045964 8) (end 21.895484 6.15048) (width 0.127) (layer "B.Cu") (net 3))
+  (segment (start 30.496499 8.10996) (end 45.99204 8.10996) (width 0.127) (layer "B.Cu") (net 3))
+  (segment (start 45.99204 8.10996) (end 46.736 7.366) (width 0.127) (layer "B.Cu") (net 3))
+  (segment (start 21.895484 6.15048) (end 28.537019 6.15048) (width 0.127) (layer "B.Cu") (net 3))
+  (segment (start 19.08 8) (end 20.045964 8) (width 0.127) (layer "B.Cu") (net 3))
+  (segment (start 28.537019 6.15048) (end 30.496499 8.10996) (width 0.127) (layer "B.Cu") (net 3))
+  (via (at 70.485 7.874) (size 0.8) (drill 0.4) (layers "F.Cu" "B.Cu") (net 4))
+  (segment (start 23.143 6.477) (end 28.40177 6.477) (width 0.127) (layer "B.Cu") (net 4))
+  (segment (start 28.40177 6.477) (end 30.36125 8.43648) (width 0.127) (layer "B.Cu") (net 4))
+  (segment (start 21.62 8) (end 23.143 6.477) (width 0.127) (layer "B.Cu") (net 4))
+  (segment (start 30.36125 8.43648) (end 69.92252 8.43648) (width 0.127) (layer "B.Cu") (net 4))
+  (segment (start 69.92252 8.43648) (end 70.485 7.874) (width 0.127) (layer "B.Cu") (net 4))
+  (via (at 93.726 8.763) (size 0.8) (drill 0.4) (layers "F.Cu" "B.Cu") (net 5))
+  (segment (start 25.273011 6.886989) (end 27.886989 6.886989) (width 0.127) (layer "B.Cu") (net 5))
+  (segment (start 28.349989 6.886989) (end 29.591 8.128) (width 0.127) (layer "B.Cu") (net 5))
+  (segment (start 29.591 8.128) (end 30.226 8.763) (width 0.127) (layer "B.Cu") (net 5))
+  (segment (start 26.238975 6.886989) (end 27.714989 6.886989) (width 0.127) (layer "B.Cu") (net 5))
+  (segment (start 30.226 8.763) (end 93.726 8.763) (width 0.127) (layer "B.Cu") (net 5))
+  (segment (start 24.16 8) (end 25.273011 6.886989) (width 0.127) (layer "B.Cu") (net 5))
+  (segment (start 27.714989 6.886989) (end 28.349989 6.886989) (width 0.127) (layer "B.Cu") (net 5))
+  (segment (start 27.7 9) (end 26.7 8) (width 0.127) (layer "F.Cu") (net 6))
+  (segment (start 29.494698 9) (end 27.7 9) (width 0.127) (layer "F.Cu") (net 6))
+  (segment (start 31.047738 7.44696) (end 29.494698 9) (width 0.127) (layer "F.Cu") (net 6))
+  (via (at 31.047738 7.44696) (size 0.8) (drill 0.4) (layers "F.Cu" "B.Cu") (net 6))
+  (zone (net 4) (net_name "TOUCH6") (layer "F.Cu") (hatch edge 0.508)
+    (priority 1)
+    (connect_pads (clearance 0.508))
+    (min_thickness 0.254) (filled_areas_thickness no)
+    (fill yes (thermal_gap 0.508) (thermal_bridge_width 0.508))
+    (polygon
+      (pts
+        (xy 96 5)
+        (xy 91 10)
+        (xy 68 10)
+        (xy 73 5)
+        (xy 68 0)
+        (xy 91 0)
+      )
+    )
+  )
   (zone (net 1) (net_name "TOUCH9") (layer "F.Cu") (hatch edge 0.508)
     (priority 1)
@@
     (polygon
       (pts
-        (xy 124 69)
-        (xy 120 73)
-        (xy 116 73)
-        (xy 116 65)
-        (xy 120 65)
-      )
-    )
-  )
-  (zone (net 6) (net_name "GND") (layers F&B.Cu) (hatch edge 0.508)
+        (xy 24 5)
+        (xy 19 10)
+        (xy 0 10)
+        (xy 0 0)
+        (xy 19 0)
+      )
+    )
+  )
+  (zone (net 2) (net_name "TOUCH8") (layer "F.Cu") (hatch edge 0.508)
+    (priority 1)
+    (connect_pads (clearance 0.508))
+    (min_thickness 0.254) (filled_areas_thickness no)
+    (fill yes (thermal_gap 0.508) (thermal_bridge_width 0.508))
+    (polygon
+      (pts
+        (xy 47 5)
+        (xy 42 10)
+        (xy 20 10)
+        (xy 25 5)
+        (xy 20 0)
+        (xy 42 0)
+      )
+    )
+  )
+  (zone (net 5) (net_name "TOUCH5") (layer "F.Cu") (hatch edge 0.508)
+    (priority 1)
+    (connect_pads (clearance 0.508))
+    (min_thickness 0.254) (filled_areas_thickness no)
+    (fill yes (thermal_gap 0.508) (thermal_bridge_width 0.508))
+    (polygon
+      (pts
+        (xy 120 10)
+        (xy 92 10)
+        (xy 97 5)
+        (xy 92 0)
+        (xy 120 0)
+      )
+    )
+  )
+  (zone (net 3) (net_name "TOUCH7") (layer "F.Cu") (hatch edge 0.508)
+    (priority 1)
+    (connect_pads (clearance 0.508))
+    (min_thickness 0.254) (filled_areas_thickness no)
+    (fill yes (thermal_gap 0.508) (thermal_bridge_width 0.508))
+    (polygon
+      (pts
+        (xy 72 5)
+        (xy 67 10)
+        (xy 43 10)
+        (xy 48 5)
+        (xy 43 0)
+        (xy 67 0)
+      )
+    )
+  )
+  (zone (net 6) (net_name "GND") (layer "B.Cu") (hatch edge 0.508)
     (connect_pads (clearance 0.508))
     (min_thickness 0.254) (filled_areas_thickness no)
@@
     (polygon
       (pts
-        (xy 171 95)
-        (xy 71 95)
-        (xy 71 50)
-        (xy 171 50)
-      )
-    )
+        (xy 120 10)
+        (xy 0 10)
+        (xy 0 0)
+        (xy 120 0)
+      )
+    )
