File: Hardware/Time-O-Mat_TouchBar/Time-O-Mat_TouchBar_H01/Time-O-Mat_TouchBar_H01.kicad_pcb (KiCad board)
At the start: 2 copper layers, 240 x 10 mm, 10 parts, among them J1 Conn_01x01_Male, J2 Conn_01x01_Male, J3 Conn_01x01_Male, J4 Conn_01x01_Male, J5 Conn_01x01_Male, J6 Conn_01x01_Male, U1 Double_Touch_Pad, U2 Double_Touch_Pad, U3 Double_Touch_Pad, U4 Double_Touch_Pad

Commit message: H01 touchbar updates
Parts:
- moved U1 24.2 mm to (18.0, 5.00)
- moved U4 10.0 mm to (222.0, 5.00)
- moved U2 3.20 mm to (81.0, 5.00)
- moved U3 0.80 mm to (159.0, 5.00)
Routing:
- net Net-(J1-Pad1): track 0.00 -> 219.7 mm, vias 0 -> 1
- net GND: track 107.4 -> 0.00 mm, vias 3 -> 0
- net Net-(J5-Pad1): track 0.00 -> 104.7 mm, vias 0 -> 1
- net Net-(J2-Pad1): track 0.00 -> 100.2 mm, vias 0 -> 1
- net Net-(J4-Pad1): track 0.00 -> 45.3 mm, vias 0 -> 1
- net Net-(J3-Pad1): track 0.00 -> 41.6 mm, vias 0 -> 1
- added copper zone on B.Cu, net GND
- removed copper zone on F.Cu, net GND
Other:
- board text added: "JLCJLCJLCJLC"
- board text added: "Time-O-Mat_TouchBar_H01"
