File: Hardware/Time-O-Mat_MoBo/Time-O-Mat_MoBo_H01/Time-O-Mat_MoBo_H01.kicad_pcb (KiCad board)
At the start: 2 copper layers, 240 x 40 mm, 79 parts, among them J1 Conn_02x04_Odd_Even, J2 Conn_02x04_Odd_Even, J3 Conn_02x04_Odd_Even, J4 Conn_02x04_Odd_Even, J5 Conn_02x04_Odd_Even, J6 Conn_01x06_Male, J7 918-418K2023S40001, J8 Conn_01x03, J9 Conn_01x05_Male, Q1 2N7002, Q2 S8050, Q3 S8050, Q4 2N7002, SW1 SW_SPST, SW2 SW_SPST, SW3 SW_SPST, SW4 SW_SPST, U1 ESP32-WROOM-32D, U2 DS18B20, U3 DS1302ZN+, U4 AMS1117-3.3, U5 CH340G, Y1 Crystal_GND2

Commit message: H01 changes
Parts:
- removed SW4: SW_SPST, Button_Switch_SMD:SW_SPST_TL3342
- added G5: Espressif_logo, Time-O-Mat_Library:Espressif_logo_30mm, F.Cu at (198.2, 36.7)
- added RESET1: SW_SPST, Button_Switch_SMD:SW_SPST_TL3342, F.Cu at (38.4, 21.2)
- C13: footprint Capacitor_SMD:C_0805_2012Metric -> Capacitor_SMD:C_0603_1608Metric
- moved G1 54.3 mm to (164.2, 33.4)
- moved R15 16.5 mm to (131.1, 21.0)
- moved R19 16.3 mm to (181.9, 27.4), turned to 90 degrees
- moved R18 14.2 mm to (179.3, 27.3), turned to 90 degrees
- moved J9 6.47 mm to (176.8, 23.7)
- moved R14 5.00 mm to (133.5, 16.8)
- moved D4 2.06 mm to (97.3, 15.0), turned to 180 degrees
- moved C11 0.40 mm to (104.6, 15.5)
- moved C13 0.30 mm to (41.0, 13.5)
Routing:
- net I2C_SDA: track 0.00 -> 159.1 mm, vias 0 -> 8
- net I2C_SCL: track 0.00 -> 148.2 mm, vias 0 -> 8
- net +3V3: track 280.2 -> 336.9 mm
- net WS2812: track 4.94 -> 31.9 mm
- net +5V: track 578.7 -> 596.6 mm, vias 7 -> 10
- net /USB+Power/ESP_RST: track 109.1 -> 125.9 mm, vias 0 -> 2
- net LIGHT2: track 80.3 -> 94.2 mm
- net Net-(J5-Pad5): track 21.9 -> 31.7 mm, vias 0 -> 2
- net GND: track 91.5 -> 99.5 mm, vias 77 -> 79
- net Net-(Q4-Pad2): track 11.6 -> 19.4 mm
- net LIGHT1: track 87.2 -> 90.7 mm
- net Net-(Q2-Pad2): track 6.48 -> 9.71 mm
- net Net-(Q3-Pad2): track 8.98 -> 12.0 mm
- net BUZZER: track 185.5 -> 187.6 mm
- net CE: track 91.6 -> 93.6 mm
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Other:
- board text added: "Electronics designed by: Marek Coufal Time-O-Mat project designed by lovely and passionate members of the Vědátoři team."
- board text added: "PCBs sponsored by Espressif."
- board text removed: "Electronics designed by: Marek Coufal Time-O-Mat project designed by lovely and supportive members of the Vědátoři team."

Commit message: H01 manufacaturing changes
Parts:
- moved G2 40.7 mm to (162.6, 34.8)
Changed lines of the file:
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@@
       (outputformat 1)
       (mirror false)
-      (drillshape 1)
+      (drillshape 0)
       (scaleselection 1)
-      (outputdirectory "")
+      (outputdirectory "Manufacturing/")
     )
   )
@@
     (fp_line (start 14.95 -2.35) (end -2.45 -2.35) (layer "F.Fab") (width 0.1))
     (fp_line (start 0 -1.35) (end 0.625 -2.35) (layer "F.Fab") (width 0.1))
-    (pad "1" thru_hole roundrect (at 0 0) (size 1.7 1.95) (drill 0.95) (layers *.Cu *.Mask) (roundrect_rratio 0.147059)
+    (pad "1" thru_hole roundrect (at 0 0) (size 1.7 1.95) (drill 0.95) (layers *.Cu *.Mask) (roundrect_rratio 0.1470588235)
       (net 18 "TOUCH9") (pinfunction "Pin_1") (pintype "passive"))
     (pad "2" thru_hole oval (at 2.5 0) (size 1.7 1.95) (drill 0.95) (layers *.Cu *.Mask)
@@
   )
   (footprint "Time-O-Mat_Library:Vedatori_copper_exposed_15mm" (layer "B.Cu")
-    (at 170 -5.2 180)
+    (at 162.56 34.798 180)
     (property "Sheetfile" "Time-O-Mat_MoBo_H01.kicad_sch")
     (property "Sheetname" "")
