File: Hardware/Time-O-Mat_MoBo/Time-O-Mat_MoBo_H01/Time-O-Mat_MoBo_H01.kicad_sch (KiCad schematic)
At the start: 54 parts, among them J1 Conn_02x04_Odd_Even, J2 Conn_02x04_Odd_Even, J3 Conn_02x04_Odd_Even, J4 Conn_02x04_Odd_Even, J5 Conn_02x04_Odd_Even, J6 Conn_01x06_Male, J8 Conn_01x03, J9 Conn_01x05_Male, Q1 2N7002, Q4 2N7002, SW1 SW_SPST, SW2 SW_SPST, SW3 SW_SPST, U1 ESP32-WROOM-32D, U2 DS18B20, U3 DS1302ZN+, Y1 Crystal_GND2

Commit message: H01 manufacaturing changes
Parts:
- added G5: (no value), symbol Time-O-Mat_Library:Espressif_logo
- C10: value (none) -> 70mF; footprint (none) -> Time-O-Mat_Library:SM3R3703T01U
- D5: value (none) -> B5819W; footprint (none) -> Diode_SMD:D_SOD-123
- G1: value CoufalElektronika_logo -> (none); footprint Time-O-Mat_Library:Coufal_elektronika_text_30x13mm -> (none)
- R16, R17: value (none) -> 1K; footprint (none) -> Resistor_SMD:R_0603_1608Metric
- R20: value (none) -> 100K; footprint (none) -> Resistor_SMD:R_0603_1608Metric
- renumbered SW4 to RESET1
Changed lines of the file:
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@@
   (symbol (lib_id "Switch:SW_SPST") (at 59.69 25.4 0) (unit 1)
     (in_bom yes) (on_board yes) (fields_autoplaced)
-    (property "Reference" "SW4" (id 0) (at 59.69 20.0492 0))
+    (property "Reference" "RESET1" (id 0) (at 59.69 20.0492 0))
     (property "Value" "" (id 1) (at 59.69 22.5861 0))
     (property "Footprint" "" (id 2) (at 59.69 25.4 0)
@@
       (effects (font (size 1.27 1.27)) (justify left))
     )
-    (property "Value" "" (id 1) (at 166.878 55.753 0)
-      (effects (font (size 1.27 1.27)) (justify left))
-    )
-    (property "Footprint" "" (id 2) (at 163.322 54.61 90)
+    (property "Value" "1K" (id 1) (at 166.878 55.753 0)
+      (effects (font (size 1.27 1.27)) (justify left))
+    )
+    (property "Footprint" "Resistor_SMD:R_0603_1608Metric" (id 2) (at 163.322 54.61 90)
       (effects (font (size 1.27 1.27)) hide)
     )
@@
     (pin "8")
   )
+  (symbol (lib_id "Time-O-Mat_Library:Espressif_logo") (at 193.04 172.72 0) (unit 1)
+    (in_bom yes) (on_board yes) (fields_autoplaced)
+    (property "Reference" "G5" (id 0) (at 193.04 170.3994 0)
+      (effects (font (size 1.27 1.27)) hide)
+    )
+    (property "Value" "" (id 1) (at 193.04 175.0406 0)
+      (effects (font (size 1.27 1.27)) hide)
+    )
+    (property "Footprint" "" (id 2) (at 193.04 172.72 0)
+      (effects (font (size 1.27 1.27)) hide)
+    )
+    (property "Datasheet" "" (id 3) (at 193.04 172.72 0)
+      (effects (font (size 1.27 1.27)) hide)
+    )
+  )
   (symbol (lib_id "Connector:Conn_01x05_Male") (at 250.19 78.74 180) (unit 1)
     (in_bom yes) (on_board yes) (fields_autoplaced)
@@
       (effects (font (size 1.27 1.27)) (justify left))
     )
-    (property "Value" "" (id 1) (at 156.718 55.753 0)
-      (effects (font (size 1.27 1.27)) (justify left))
-    )
-    (property "Footprint" "" (id 2) (at 153.162 54.61 90)
+    (property "Value" "1K" (id 1) (at 156.718 55.753 0)
+      (effects (font (size 1.27 1.27)) (justify left))
+    )
+    (property "Footprint" "Resistor_SMD:R_0603_1608Metric" (id 2) (at 153.162 54.61 90)
       (effects (font (size 1.27 1.27)) hide)
     )
@@
       (effects (font (size 1.27 1.27)) (justify left))
     )
-    (property "Value" "" (id 1) (at 276.86 138.43 0)
-      (effects (font (size 1.27 1.27)) (justify left))
-    )
-    (property "Footprint" "" (id 2) (at 277.8252 148.59 0)
+    (property "Value" "70mF" (id 1) (at 276.86 138.43 0)
+      (effects (font (size 1.27 1.27)) (justify left))
+    )
+    (property "Footprint" "Time-O-Mat_Library:SM3R3703T01U" (id 2) (at 277.8252 148.59 0)
       (effects (font (size 1.27 1.27)) hide)
     )
@@
       (effects (font (size 1.27 1.27)) (justify left))
     )
-    (property "Value" "" (id 1) (at 278.638 126.873 0)
-      (effects (font (size 1.27 1.27)) (justify left))
-    )
-    (property "Footprint" "" (id 2) (at 275.082 125.73 90)
+    (property "Value" "100K" (id 1) (at 278.638 126.873 0)
+      (effects (font (size 1.27 1.27)) (justify left))
+    )
+    (property "Footprint" "Resistor_SMD:R_0603_1608Metric" (id 2) (at 275.082 125.73 90)
       (effects (font (size 1.27 1.27)) hide)
     )
@@
       (effects (font (size 1.27 1.27)) hide)
     )
-    (property "Value" "CoufalElektronika_logo" (id 1) (at 223.52 180.8512 0)
-      (effects (font (size 1.27 1.27)) hide)
-    )
-    (property "Footprint" "Time-O-Mat_Library:Coufal_elektronika_text_30x13mm" (id 2) (at 223.52 173.99 0)
+    (property "Value" "" (id 1) (at 223.52 180.8512 0)
+      (effects (font (size 1.27 1.27)) hide)
+    )
+    (property "Footprint" "" (id 2) (at 223.52 173.99 0)
       (effects (font (size 1.27 1.27)) hide)
     )
@@
       (effects (font (size 1.27 1.27)) (justify left))
     )
-    (property "Value" "" (id 1) (at 274.828 116.967 90)
-      (effects (font (size 1.27 1.27)) (justify left))
-    )
-    (property "Footprint" "" (id 2) (at 276.86 118.11 0)
+    (property "Value" "B5819W" (id 1) (at 274.828 116.967 90)
+      (effects (font (size 1.27 1.27)) (justify left))
+    )
+    (property "Footprint" "Diode_SMD:D_SOD-123" (id 2) (at 276.86 118.11 0)
       (effects (font (size 1.27 1.27)) hide)
     )
@@
     )
     (path "/4ec8e228-d742-4cd8-8c0d-36879b06f45c/1e8d74aa-646d-4bbb-b7d1-3adf29d77062"
-      (reference "C13") (unit 1) (value "10u") (footprint "Capacitor_SMD:C_0805_2012Metric")
+      (reference "C13") (unit 1) (value "10u") (footprint "Capacitor_SMD:C_0603_1608Metric")
     )
     (path "/4ec8e228-d742-4cd8-8c0d-36879b06f45c/32bd4d0c-de0e-4075-bccf-c1fd4cbc1177"
@@
       (reference "G3") (unit 1) (value "Vedatori_logo") (footprint "Time-O-Mat_Library:Vedatori_15mm")
     )
+    (path "/540a2e69-fa71-4298-a5af-e20a2aa565c0"
+      (reference "G5") (unit 1) (value "Espressif_logo") (footprint "Time-O-Mat_Library:Espressif_logo_30mm")
+    )
     (path "/9166ea7b-5cf9-4faf-8e58-cdcf7a4c35af"
       (reference "H1") (unit 1) (value "MountingHole") (footprint "MountingHole:MountingHole_3.2mm_M3")
@@
       (reference "R20") (unit 1) (value "100K") (footprint "Resistor_SMD:R_0603_1608Metric")
     )
+    (path "/0e23d0bb-eccc-4885-8a3e-8730a3f991e0"
+      (reference "RESET1") (unit 1) (value "SW_SPST") (footprint "Button_Switch_SMD:SW_SPST_TL3342")
+    )
     (path "/350b7ccb-1ee9-421d-93df-bf4125243817"
       (reference "SW1") (unit 1) (value "SW_SPST") (footprint "Button_Switch_THT:SW_Tactile_SPST_Angled_PTS645Vx83-2LFS")
@@
       (reference "SW3") (unit 1) (value "SW_SPST") (footprint "Button_Switch_THT:SW_Tactile_SPST_Angled_PTS645Vx83-2LFS")
     )
-    (path "/0e23d0bb-eccc-4885-8a3e-8730a3f991e0"
-      (reference "SW4") (unit 1) (value "SW_SPST") (footprint "Button_Switch_SMD:SW_SPST_TL3342")
-    )
     (path "/4ec8e228-d742-4cd8-8c0d-36879b06f45c/98b95900-32c2-49ce-8dc5-9c732767bfd5"
