File: Hardware/Time-O-Mat_MoBo/Time-O-Mat_MoBo_H01/USB+Power.kicad_sch (KiCad schematic)
At the start: 23 parts, among them J7 918-418K2023S40001, Q2 S8050, Q3 S8050, U4 AMS1117-3.3, U5 CH340G

Commit message: H01 manufacaturing changes
Parts:
- C13: value 10u -> (none); footprint Capacitor_SMD:C_0805_2012Metric -> (none); LCSC C15850 -> C19702
Changed lines of the file:
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@@
       (effects (font (size 1.27 1.27)) (justify left))
     )
-    (property "Value" "10u" (id 1) (at 115.951 65.913 0)
+    (property "Value" "" (id 1) (at 115.951 65.913 0)
       (effects (font (size 1.27 1.27)) (justify left))
     )
-    (property "Footprint" "Capacitor_SMD:C_0805_2012Metric" (id 2) (at 113.9952 68.58 0)
+    (property "Footprint" "" (id 2) (at 113.9952 68.58 0)
       (effects (font (size 1.27 1.27)) hide)
     )
@@
       (effects (font (size 1.27 1.27)) hide)
     )
-    (property "LCSC" "C15850" (id 4) (at 113.03 64.77 0)
+    (property "LCSC" "C19702" (id 4) (at 113.03 64.77 0)
       (effects (font (size 1.27 1.27)) hide)
     )
