File: Hardware/Time-O-Mat_MoBo/Time-O-Mat_MoBo_H02/Time-O-Mat_MoBo_H02.kicad_pcb (KiCad board)
At the start: 2 copper layers, 240 x 40 mm, 86 parts, among them J1 Conn_02x04_Odd_Even, J2 Conn_02x04_Odd_Even, J3 Conn_02x04_Odd_Even, J4 Conn_02x04_Odd_Even, J5 Conn_02x04_Odd_Even, J6 Conn_01x06_Male, J7 918-418K2023S40001, J8 Conn_01x03, J9 Conn_01x05_Male, Q1 2N7002, Q2 S8050, Q3 S8050, Q4 2N7002, SW1 SW_SPST, SW2 SW_SPST, SW3 SW_SPST, U1 ESP32-WROOM-32D, U2 DS18B20, U3 DS1302ZN+, U4 AMS1117-3.3, U5 CH340G, Y1 Crystal_GND2

Commit message: H02 updates
Parts:
- moved C7 4.62 mm to (201.9, 11.6), turned to 180 degrees
Routing:
- net +5V: track 596.6 -> 587.2 mm
- net +3V3: track 336.8 -> 340.4 mm
- net GND: track 102.7 -> 104.7 mm, vias 81 -> 80
Other:
- board text added: "Time-O-Mat_Mobo_H02 12.07.2022"
- board text removed: "Time-O-Mat_Mobo_H01"
