File: Hardware/Time-O-Mat_MoBo/Time-O-Mat_MoBo_H02/Time-O-Mat_MoBo_H02.kicad_pcb (KiCad board)
At the start: 2 copper layers, 240 x 40 mm, 86 parts, among them J1 Conn_02x04_Odd_Even, J2 Conn_02x04_Odd_Even, J3 Conn_02x04_Odd_Even, J4 Conn_02x04_Odd_Even, J5 Conn_02x04_Odd_Even, J6 Conn_01x06_Male, J7 918-418K2023S40001, J8 Conn_01x03, J9 Conn_01x05_Male, Q1 2N7002, Q2 S8050, Q3 S8050, Q4 2N7002, SW1 SW_SPST, SW2 SW_SPST, SW3 SW_SPST, U1 ESP32-WROOM-32D, U2 DS18B20, U3 DS1302ZN+, U4 AMS1117-3.3, U5 CH340G, Y1 Crystal_GND2

Commit message: H02 changes
Parts:
- moved C15 2.00 mm to (117.6, 9.56)
- moved R13 2.00 mm to (121.0, 9.56)
- moved R21 2.00 mm to (119.3, 9.56)
- moved R12 1.96 mm to (113.6, 8.00)
Routing:
- net LIGHT1: track 84.6 -> 86.9 mm
- net +3V3: track 340.4 -> 342.4 mm
- net Net-(R12-Pad2): track 12.6 -> 14.5 mm
- net GND: track 104.7 -> 105.2 mm
Other:
- board text added: "GND SCL SDA 3V3 5V"
