File: Hardware/Time-O-Mat_MoBo/Time-O-Mat_MoBo_H02/Time-O-Mat_MoBo_H02.kicad_sch (KiCad schematic)
At the start: 55 parts, among them J1 Conn_02x04_Odd_Even, J2 Conn_02x04_Odd_Even, J3 Conn_02x04_Odd_Even, J4 Conn_02x04_Odd_Even, J5 Conn_02x04_Odd_Even, J6 Conn_01x06_Male, J8 Conn_01x03, J9 Conn_01x05_Male, Q1 2N7002, Q4 2N7002, SW1 SW_SPST, SW2 SW_SPST, SW3 SW_SPST, U1 ESP32-WROOM-32D, U2 DS18B20, U3 DS1302ZN+, Y1 Crystal_GND2

Commit message: H02 updates
Parts:
- added C15, C17: 1u, Capacitor_SMD:C_0603_1608Metric, symbol Device:C
- added R21, R22: 100K, Resistor_SMD:R_0603_1608Metric, symbol Device:R
- G2: value Vedatori_logo -> (none); footprint Time-O-Mat_Library:Vedatori_copper_exposed_15mm -> (none)
- J8: footprint (none) -> Connector_JST:JST_XH_S3B-XH-A-1_1x03_P2.50mm_Horizontal
- R12: footprint (none) -> Connector_JST:JST_XH_S2B-XH-A-1_1x02_P2.50mm_Horizontal
- R20: value 100K -> (none); footprint Resistor_SMD:R_0603_1608Metric -> (none); LCSC C25803 -> C22859
Connections:
- net GND: now also C15.1, C17.1
- net LIGHT1: now also C15.2, R21.2; no longer R12.2, R13.1
- net LIGHT2: now also C17.2, R22.2; no longer R14.2, R15.1
- new net: R14.2, R15.1, R22.1
- new net: R12.2, R13.1, R21.1
Other:
- moved on the sheet: R12, R13, R14, R15
