File: Hardware/Time-O-Mat_MoBo/Time-O-Mat_MoBo_H02/USB+Power.kicad_sch (KiCad schematic)
At the start: 23 parts, among them J7 918-418K2023S40001, Q2 S8050, Q3 S8050, U4 AMS1117-3.3, U5 CH340G

Commit message: H02 updates
Parts:
- added R23, R24: 100K, Resistor_SMD:R_0603_1608Metric, symbol Device:R
Connections:
- net CC1: now also R23.2; no longer J7.A5 (CC1), R5.2
- net CC2: now also R24.2; no longer J7.B5 (CC2), R7.2
- new net: J7.A5 (CC1), R23.1, R5.2
- new net: J7.B5 (CC2), R24.1, R7.2
Other:
- moved on the sheet: R5, R7
Changed lines of the file:
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@@
 (kicad_sch (version 20211123) (generator eeschema)
   (paper "A4")
+  (junction (at 83.82 63.5) (diameter 0) (color 0 0 0 0)
+  )
   (junction (at 113.03 128.27) (diameter 0) (color 0 0 0 0)
   )
@@
   )
   (junction (at 78.74 73.66) (diameter 0) (color 0 0 0 0)
+  )
+  (junction (at 93.98 66.04) (diameter 0) (color 0 0 0 0)
   )
   (no_connect (at 129.54 68.58))
@@
   (no_connect (at 149.86 76.2))
   (no_connect (at 149.86 73.66))
-  (wire (pts (xy 93.98 66.04) (xy 93.98 64.77))
+  (wire (pts (xy 93.98 66.04) (xy 93.98 48.26))
     (stroke (width 0) (type default) (color 0 0 0 0))
   )
@@
     (stroke (width 0) (type default) (color 0 0 0 0))
   )
-  (wire (pts (xy 83.82 64.77) (xy 78.74 64.77))
+  (wire (pts (xy 83.82 48.26) (xy 83.82 63.5))
     (stroke (width 0) (type default) (color 0 0 0 0))
   )
@@
     (stroke (width 0) (type default) (color 0 0 0 0))
   )
-  (wire (pts (xy 78.74 64.77) (xy 78.74 63.5))
+  (wire (pts (xy 83.82 63.5) (xy 78.74 63.5))
     (stroke (width 0) (type default) (color 0 0 0 0))
   )
@@
     (effects (font (size 1.27 1.27)) (justify left bottom))
   )
-  (global_label "CC1" (shape input) (at 83.82 64.77 0) (fields_autoplaced)
+  (global_label "CC1" (shape input) (at 91.44 63.5 90) (fields_autoplaced)
     (effects (font (size 1.27 1.27)) (justify left))
-    (property "Intersheet References" "${INTERSHEET_REFS}" (id 0) (at 89.9826 64.6906 0)
+    (property "Intersheet References" "${INTERSHEET_REFS}" (id 0) (at 91.3606 57.3374 90)
       (effects (font (size 1.27 1.27)) (justify left) hide)
     )
   )
-  (global_label "CC2" (shape input) (at 93.98 66.04 0) (fields_autoplaced)
+  (global_label "CC2" (shape input) (at 101.6 66.04 0) (fields_autoplaced)
     (effects (font (size 1.27 1.27)) (justify left))
-    (property "Intersheet References" "${INTERSHEET_REFS}" (id 0) (at 100.1426 65.9606 0)
+    (property "Intersheet References" "${INTERSHEET_REFS}" (id 0) (at 107.7626 65.9606 0)
       (effects (font (size 1.27 1.27)) (justify left) hide)
     )
@@
     (pin "2")
   )
-  (symbol (lib_id "power:GND") (at 83.82 57.15 180) (unit 1)
-    (in_bom yes) (on_board yes)
-    (property "Reference" "#PWR0159" (id 0) (at 83.82 50.8 0)
-      (effects (font (size 1.27 1.27)) hide)
-    )
-    (property "Value" "GND" (id 1) (at 83.693 52.7558 0))
-    (property "Footprint" "" (id 2) (at 83.82 57.15 0)
-      (effects (font (size 1.27 1.27)) hide)
-    )
-    (property "Datasheet" "" (id 3) (at 83.82 57.15 0)
+  (symbol (lib_id "power:GND") (at 83.82 40.64 180) (unit 1)
+    (in_bom yes) (on_board yes)
+    (property "Reference" "#PWR0159" (id 0) (at 83.82 34.29 0)
+      (effects (font (size 1.27 1.27)) hide)
+    )
+    (property "Value" "GND" (id 1) (at 83.693 36.2458 0))
+    (property "Footprint" "" (id 2) (at 83.82 40.64 0)
+      (effects (font (size 1.27 1.27)) hide)
+    )
+    (property "Datasheet" "" (id 3) (at 83.82 40.64 0)
       (effects (font (size 1.27 1.27)) hide)
     )
@@
     (pin "1")
   )
+  (symbol (lib_id "Device:R") (at 97.79 66.04 90) (unit 1)
+    (in_bom yes) (on_board yes)
+    (property "Reference" "R24" (id 0) (at 96.6216 64.262 0)
+      (effects (font (size 1.27 1.27)) (justify left))
+    )
+    (property "Value" "100K" (id 1) (at 98.933 64.262 0)
+      (effects (font (size 1.27 1.27)) (justify left))
+    )
+    (property "Footprint" "Resistor_SMD:R_0603_1608Metric" (id 2) (at 97.79 67.818 90)
+      (effects (font (size 1.27 1.27)) hide)
+    )
+    (property "Datasheet" "~" (id 3) (at 97.79 66.04 0)
+      (effects (font (size 1.27 1.27)) hide)
+    )
+    (property "LCSC" "C25803" (id 4) (at 97.79 66.04 0)
+      (effects (font (size 1.27 1.27)) hide)
+    )
+    (pin "1")
+    (pin "2")
+  )
   (symbol (lib_id "Device:Q_NPN_BEC") (at 179.07 96.52 0) (mirror x) (unit 1)
     (in_bom yes) (on_board yes)
@@
     (pin "2")
   )
-  (symbol (lib_id "power:GND") (at 93.98 57.15 180) (unit 1)
-    (in_bom yes) (on_board yes)
-    (property "Reference" "#PWR0158" (id 0) (at 93.98 50.8 0)
-      (effects (font (size 1.27 1.27)) hide)
-    )
-    (property "Value" "GND" (id 1) (at 93.853 52.7558 0))
-    (property "Footprint" "" (id 2) (at 93.98 57.15 0)
-      (effects (font (size 1.27 1.27)) hide)
-    )
-    (property "Datasheet" "" (id 3) (at 93.98 57.15 0)
+  (symbol (lib_id "power:GND") (at 93.98 40.64 180) (unit 1)
+    (in_bom yes) (on_board yes)
+    (property "Reference" "#PWR0158" (id 0) (at 93.98 34.29 0)
+      (effects (font (size 1.27 1.27)) hide)
+    )
+    (property "Value" "GND" (id 1) (at 93.853 36.2458 0))
+    (property "Footprint" "" (id 2) (at 93.98 40.64 0)
+      (effects (font (size 1.27 1.27)) hide)
+    )
+    (property "Datasheet" "" (id 3) (at 93.98 40.64 0)
       (effects (font (size 1.27 1.27)) hide)
     )
@@
     (pin "2")
   )
-  (symbol (lib_id "Device:R") (at 83.82 60.96 0) (unit 1)
-    (in_bom yes) (on_board yes)
-    (property "Reference" "R5" (id 0) (at 85.598 59.7916 0)
-      (effects (font (size 1.27 1.27)) (justify left))
-    )
-    (property "Value" "5K1" (id 1) (at 85.598 62.103 0)
-      (effects (font (size 1.27 1.27)) (justify left))
-    )
-    (property "Footprint" "Resistor_SMD:R_0603_1608Metric" (id 2) (at 82.042 60.96 90)
-      (effects (font (size 1.27 1.27)) hide)
-    )
-    (property "Datasheet" "~" (id 3) (at 83.82 60.96 0)
-      (effects (font (size 1.27 1.27)) hide)
-    )
-    (property "LCSC" "C23186" (id 4) (at 83.82 60.96 0)
+  (symbol (lib_id "Device:R") (at 83.82 44.45 0) (unit 1)
+    (in_bom yes) (on_board yes)
+    (property "Reference" "R5" (id 0) (at 85.598 43.2816 0)
+      (effects (font (size 1.27 1.27)) (justify left))
+    )
+    (property "Value" "5K1" (id 1) (at 85.598 45.593 0)
+      (effects (font (size 1.27 1.27)) (justify left))
+    )
+    (property "Footprint" "Resistor_SMD:R_0603_1608Metric" (id 2) (at 82.042 44.45 90)
+      (effects (font (size 1.27 1.27)) hide)
+    )
+    (property "Datasheet" "~" (id 3) (at 83.82 44.45 0)
+      (effects (font (size 1.27 1.27)) hide)
+    )
+    (property "LCSC" "C23186" (id 4) (at 83.82 44.45 0)
       (effects (font (size 1.27 1.27)) hide)
     )
@@
     (pin "2")
   )
-  (symbol (lib_id "Device:R") (at 93.98 60.96 0) (unit 1)
-    (in_bom yes) (on_board yes)
-    (property "Reference" "R7" (id 0) (at 95.758 59.7916 0)
-      (effects (font (size 1.27 1.27)) (justify left))
-    )
-    (property "Value" "5K1" (id 1) (at 95.758 62.103 0)
-      (effects (font (size 1.27 1.27)) (justify left))
-    )
-    (property "Footprint" "Resistor_SMD:R_0603_1608Metric" (id 2) (at 92.202 60.96 90)
-      (effects (font (size 1.27 1.27)) hide)
-    )
-    (property "Datasheet" "~" (id 3) (at 93.98 60.96 0)
-      (effects (font (size 1.27 1.27)) hide)
-    )
-    (property "LCSC" "C23186" (id 4) (at 93.98 60.96 0)
+  (symbol (lib_id "Device:R") (at 93.98 44.45 0) (unit 1)
+    (in_bom yes) (on_board yes)
+    (property "Reference" "R7" (id 0) (at 95.758 43.2816 0)
+      (effects (font (size 1.27 1.27)) (justify left))
+    )
+    (property "Value" "5K1" (id 1) (at 95.758 45.593 0)
+      (effects (font (size 1.27 1.27)) (justify left))
+    )
+    (property "Footprint" "Resistor_SMD:R_0603_1608Metric" (id 2) (at 92.202 44.45 90)
+      (effects (font (size 1.27 1.27)) hide)
+    )
+    (property "Datasheet" "~" (id 3) (at 93.98 44.45 0)
+      (effects (font (size 1.27 1.27)) hide)
+    )
+    (property "LCSC" "C23186" (id 4) (at 93.98 44.45 0)
       (effects (font (size 1.27 1.27)) hide)
     )
@@
       (effects (font (size 1.27 1.27)) hide)
     )
+    (pin "1")
+    (pin "2")
+  )
+  (symbol (lib_id "Device:R") (at 87.63 63.5 90) (unit 1)
+    (in_bom yes) (on_board yes)
+    (property "Reference" "R23" (id 0) (at 86.4616 61.722 0)
+      (effects (font (size 1.27 1.27)) (justify left))
+    )
+    (property "Value" "100K" (id 1) (at 88.773 61.722 0)
+      (effects (font (size 1.27 1.27)) (justify left))
+    )
+    (property "Footprint" "Resistor_SMD:R_0603_1608Metric" (id 2) (at 87.63 65.278 90)
+      (effects (font (size 1.27 1.27)) hide)
+    )
+    (property "Datasheet" "~" (id 3) (at 87.63 63.5 0)
+      (effects (font (size 1.27 1.27)) hide)
+    )
+    (property "LCSC" "C25803" (id 4) (at 87.63 63.5 0)
+      (effects (font (size 1.27 1.27)) hide)
+    )
